File: faceplates/pulp-logic-1u-faceplate-6hp/pulp-logic-1u-faceplate-6hp.kicad_pcb (KiCad board)
At the start: 2 copper layers, 30 x 43.2 mm, 2 parts

Commit message: Moving mounting holes
Parts:
- moved REF** 2.42 mm to (5.08, 40.2)
- moved REF** 2.42 mm to (5.08, 3.00)
Changed lines of the file:
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@@
   (net 0 "")
   (footprint "MountingHole:MountingHole_3.2mm_M3" (layer "F.Cu")
-    (at 7.5 40.2)
+    (at 5.08 40.2)
     (descr "Mounting Hole 3.2mm, no annular, M3")
     (tags "mounting hole 3.2mm no annular m3")
@@
   )
   (footprint "MountingHole:MountingHole_3.2mm_M3" (layer "F.Cu")
-    (at 7.5 3)
+    (at 5.08 3)
     (descr "Mounting Hole 3.2mm, no annular, M3")
     (tags "mounting hole 3.2mm no annular m3")
